Commit message: modified shadowhand

File: data/ShadowHand/shadowhand.urdf (robot description, URDF)
Before this commit: robot shadowhand, 28 links, 27 joints
Links:
- removed link fftip
- removed link lftip
- removed link mftip
- removed link rftip
- removed link thtip
- link thbase: geometry collision box size=0.1 0.1 0.1; visual box size=0.001 0.001 0.001
Joints:
- removed joint FFtip
- removed joint LFtip
- removed joint MFtip
- removed joint RFtip
- removed joint thtip

Commit message: upgraded shadowhand

File: data/ShadowHand/shadowhand.urdf (robot description, URDF)
Before this commit: robot shadowhand, 23 links, 22 joints
Links:
- added link fftip, mass 0.001
- added link forearm, mass 3.0; collision cylinder length=0.180 radius=0.06; visual mesh filename=meshes/forearm.obj scale=0.1 0.1 0.1
- added link lftip, mass 0.001
- added link mftip, mass 0.001
- added link rftip, mass 0.001
- added link thtip, mass 0.001
- added link wrist, mass 0.1; collision box size=0.02 0.02 0.02; visual mesh filename=meshes/wrist.obj scale=0.1 0.1 0.1
- link ffdistal: geometry collision mesh filename=meshes/distal_ellipsoid.obj scale=0.1 0.1 0.1; visual mesh filename=meshes/distal_ellipsoid.obj scale=0.1 0.1 0.1
- link ffknuckle: geometry collision box size=0.005 0.005 0.005; visual mesh filename=meshes/knuckle.obj scale=0.1 0.1 0.1
- link ffmiddle: geometry collision box size=0.008 0.008 0.015; visual mesh filename=meshes/F2.obj scale=0.1 0.1 0.1
- link ffproximal: geometry collision box size=0.008 0.008 0.04; visual mesh filename=meshes/F3.obj scale=0.1 0.1 0.1
- link lfdistal: geometry collision mesh filename=meshes/F1.obj scale=0.1 0.1 0.1; visual mesh filename=meshes/F1.obj scale=0.1 0.1 0.1
- link lfknuckle: geometry collision box size=0.005 0.005 0.005; visual mesh filename=meshes/knuckle.obj scale=0.1 0.1 0.1
- link lfmetacarpal: geometry collision box size=0.008 0.008 0.03; visual mesh filename=meshes/lfmetacarpal.obj scale=0.1 0.1 0.1
- link lfmiddle: geometry collision box size=0.008 0.008 0.015; visual mesh filename=meshes/F2.obj scale=0.1 0.1 0.1
- link lfproximal: geometry collision box size=0.008 0.008 0.04; visual mesh filename=meshes/F3.obj scale=0.1 0.1 0.1
- link mfdistal: geometry collision mesh filename=meshes/F1.obj scale=0.1 0.1 0.1; visual mesh filename=meshes/F1.obj scale=0.1 0.1 0.1
- link mfknuckle: geometry collision box size=0.005 0.005 0.005; visual mesh filename=meshes/knuckle.obj scale=0.1 0.1 0.1
- link mfmiddle: geometry collision box size=0.008 0.008 0.015; visual mesh filename=meshes/F2.obj scale=0.1 0.1 0.1
- link mfproximal: geometry collision box size=0.008 0.008 0.04; visual mesh filename=meshes/F3.obj scale=0.1 0.1 0.1
- link palm: geometry collision box size=0.05 0.02 0.07; visual mesh filename=meshes/palm.obj scale=0.1 0.1 0.1
- link rfdistal: geometry collision mesh filename=meshes/distal_ellipsoid.obj scale=0.1 0.1 0.1; visual mesh filename=meshes/distal_ellipsoid.obj scale=0.1 0.1 0.1
- link rfknuckle: geometry collision box size=0.005 0.005 0.005; visual mesh filename=meshes/knuckle.obj scale=0.1 0.1 0.1
- link rfmiddle: geometry collision box size=0.008 0.008 0.015; visual mesh filename=meshes/F2.obj scale=0.1 0.1 0.1
- link rfproximal: geometry collision box size=0.008 0.008 0.04; visual mesh filename=meshes/F3.obj scale=0.1 0.1 0.1
- link thbase: geometry collision box size=0.001 0.001 0.001; visual box size=0.001 0.001 0.001
- link thdistal: geometry collision mesh filename=meshes/distal_ellipsoid.obj scale=0.1 0.1 0.1; visual mesh filename=meshes/distal_ellipsoid.obj scale=0.1 0.1 0.1
- link thmiddle: geometry collision box size=0.008 0.008 0.015; visual mesh filename=meshes/TH2_z.obj scale=0.1 0.1 0.1
- link thproximal: geometry collision box size=0.008 0.008 0.020; visual mesh filename=meshes/TH3_z.obj scale=0.1 0.1 0.1
Joints:
- added joint FFtip: type fixed, parent ffdistal, child fftip, origin xyz=0 0 0.026 rpy=0 0 0
- added joint LFtip: type fixed, parent lfdistal, child lftip, origin xyz=0 0 0.026 rpy=0 0 0
- added joint MFtip: type fixed, parent mfdistal, child mftip, origin xyz=0 0 0.026 rpy=0 0 0
- added joint RFtip: type fixed, parent rfdistal, child rftip, origin xyz=0 0 0.026 rpy=0 0 0
- added joint WRJ1: type revolute, parent wrist, child palm, origin xyz=0 0 0.034 rpy=0 0 0, axis 1 0 0, limit lower=-0.78539816339744828 upper=0.6108652381980153 effort=5 velocity=1.0
- added joint WRJ2: type revolute, parent forearm, child wrist, origin xyz=0 -0.010 0.213 rpy=0 0 0, axis 0 1 0, limit lower=-0.52359877559829882 upper=0.17453292519943295 effort=5 velocity=1.0
- added joint thtip: type fixed, parent thdistal, child thtip, origin xyz=0 0 0.0275 rpy=0 0 0
